File: PCB/devboard.kicad_sch (KiCad schematic)
At the start: 32 parts, among them J1 USB_C_Receptacle_USB2.0_14P, J2 Conn_01x20, J3 Conn_01x20, J4 Conn_01x03, SW1 SW_Push, U1 RP2040, U2 MCP1700x-330xxTT, U3 W25Q16JVUXIQ TR, Y1 Crystal_GND24

Commit message: updating readme and pcb
Other:
- note added: "FredBoard"
- note added: "Made by Mary"
- moved on the sheet: C13, C14, J1, J2, J3, J4, R1, R2, R3, R4, U1, U2
