File: v1/PCB/devboard.kicad_sch (KiCad schematic)
At the start: 36 parts, among them J1 USB_C_Receptacle_USB2.0_14P, J2 Conn_01x20, J3 Conn_01x20, J4 Conn_01x03, SW1 SW_Push, U1 RP2040, U2 MCP1700x-330xxTT, U3 W25Q16JVUXIQ TR, Y1 Crystal_GND24

Commit message: updated pcb and made renders
-Changed imu to a MPU-6500
-moved some traces and changed some pads in the devboard
-remade gerber and BOM
-created renders of the v2
-made pinout image of the v2
Parts:
- R9: value 1K -> 150
Connections:
- net +3.3V: now also R8.2; no longer R8.1
- net at D1.2 (A): now also R8.1; no longer R8.2
Other:
- moved on the sheet: R8
Changed lines of the file:
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@@
 	(wire
 		(pts
-			(xy 101.6 31.75) (xy 101.6 44.45)
+			(xy 101.6 31.75) (xy 101.6 43.18)
 		)
 		(stroke
@@
 	(wire
 		(pts
-			(xy 100.33 50.8) (xy 101.6 50.8)
-		)
-		(stroke
-			(width 0)
-			(type default)
-		)
-	)
-	(wire
-		(pts
 			(xy 76.2 31.75) (xy 78.74 31.75)
 		)
@@
 	(wire
 		(pts
-			(xy 92.71 44.45) (xy 92.71 50.8)
-		)
-		(stroke
-			(width 0)
-			(type default)
-		)
-	)
-	(wire
-		(pts
 			(xy 187.96 114.3) (xy 186.69 114.3)
 		)
@@
 	(wire
 		(pts
-			(xy 101.6 44.45) (xy 92.71 44.45)
-		)
-		(stroke
-			(width 0)
-			(type default)
-		)
-	)
-	(wire
-		(pts
 			(xy 86.36 153.67) (xy 86.36 166.37)
 		)
@@
 			)
 		)
-		(property "Value" "1K"
+		(property "Value" "150"
 			(at 211.074 152.654 90)
 			(show_name no)
@@
 	(symbol
 		(lib_id "Device:R")
-		(at 96.52 50.8 90)
+		(at 101.6 46.99 180)
 		(unit 1)
 		(body_style 1)
@@
 		(fields_autoplaced yes)
 		(property "Reference" "R8"
-			(at 96.52 44.45 90)
+			(at 104.14 45.7199 0)
 			(show_name no)
 			(do_not_autoplace no)
@@
 					(size 1.27 1.27)
 				)
+				(justify right)
 			)
 		)
 		(property "Value" "1K"
-			(at 96.52 46.99 90)
+			(at 104.14 48.2599 0)
 			(show_name no)
 			(do_not_autoplace no)
@@
 					(size 1.27 1.27)
 				)
+				(justify right)
 			)
 		)
 		(property "Footprint" "Resistor_SMD:R_0402_1005Metric"
-			(at 96.52 52.578 90)
+			(at 103.378 46.99 90)
 			(hide yes)
 			(show_name no)
@@
 		)
 		(property "Datasheet" ""
-			(at 96.52 50.8 0)
+			(at 101.6 46.99 0)
 			(hide yes)
 			(show_name no)
@@
 		)
 		(property "Description" "Resistor"
-			(at 96.52 50.8 0)
+			(at 101.6 46.99 0)
 			(hide yes)
 			(show_name no)
