File: v1/PCB/devboard.kicad_pcb (KiCad board)
At the start: 2 copper layers, 51 x 21 mm, 36 parts, among them J1 USB_C_Receptacle_USB2.0_14P, J2 Conn_01x20, J3 Conn_01x20, J4 Conn_01x03, SW1 SW_Push, U1 RP2040, U2 MCP1700x-330xxTT, U3 W25Q16JVUXIQ TR, Y1 Crystal_GND24

Commit message: updated pcb and made renders
-Changed imu to a MPU-6500
-moved some traces and changed some pads in the devboard
-remade gerber and BOM
-created renders of the v2
-made pinout image of the v2
Parts:
- R9: value 1K -> 150
Connections:
- R8 pad 1: +3.3V -> Net-(D1-A)
- R8 pad 2: Net-(D1-A) -> +3.3V
Changed lines of the file:
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@@
 			(layers "F.Cu" "F.Mask" "F.Paste")
 			(roundrect_rratio 0.25)
-			(net "+3.3V")
+			(net "Net-(D1-A)")
 			(pintype "passive")
 		)
@@
 			(layers "F.Cu" "F.Mask" "F.Paste")
 			(roundrect_rratio 0.25)
-			(net "Net-(D1-A)")
+			(net "+3.3V")
 			(pintype "passive")
 		)
@@
 			)
 		)
-		(property "Value" "1K"
+		(property "Value" "150"
 			(at 0 1.17 0)
 			(layer "F.Fab")
@@
 	)
 	(segment
+		(start 105.3338 63.2992)
+		(end 105.3314 63.2968)
+		(width 0.2)
+		(layer "F.Cu")
+		(net "Net-(D1-A)")
+	)
+	(segment
+		(start 105.3338 64.3342)
+		(end 105.3338 63.2992)
+		(width 0.2)
+		(layer "F.Cu")
+		(net "Net-(D1-A)")
+	)
+	(segment
 		(start 108.655 70.4068)
 		(end 107.6878 71.374)
@@
 	)
 	(segment
+		(start 129.0614 65.405)
+		(end 130.2028 65.405)
+		(width 0.2)
+		(layer "F.Cu")
+		(net "Net-(D2-A)")
+	)
+	(segment
+		(start 130.2028 65.405)
+		(end 130.3274 65.5296)
+		(width 0.2)
+		(layer "F.Cu")
+		(net "Net-(D2-A)")
+	)
+	(segment
+		(start 118.0556 64.9442)
+		(end 118.0592 64.9478)
+		(width 0.2)
+		(layer "F.Cu")
+		(net "led2")
+	)
+	(segment
+		(start 128.0414 65.405)
+		(end 127 65.405)
+		(width 0.2)
+		(layer "F.Cu")
+		(net "led2")
+	)
+	(segment
+		(start 118.0556 64.0757)
+		(end 118.0556 64.9442)
+		(width 0.2)
+		(layer "F.Cu")
+		(net "led2")
+	)
+	(segment
+		(start 127 65.405)
+		(end 126.7206 65.6844)
+		(width 0.2)
+		(layer "F.Cu")
+		(net "led2")
+	)
+	(via
+		(at 126.7206 65.6844)
+		(size 0.6)
+		(drill 0.3)
+		(layers "F.Cu" "B.Cu")
+		(net "led2")
+	)
+	(via
+		(at 118.0592 64.9478)
+		(size 0.6)
+		(drill 0.3)
+		(layers "F.Cu" "B.Cu")
+		(net "led2")
+	)
+	(segment
+		(start 126.3714 66.0336)
+		(end 126.7206 65.6844)
+		(width 0.2)
+		(layer "B.Cu")
+		(net "led2")
+	)
+	(segment
+		(start 119.145 66.0336)
+		(end 126.3714 66.0336)
+		(width 0.2)
+		(layer "B.Cu")
+		(net "led2")
+	)
+	(segment
+		(start 118.0592 64.9478)
+		(end 119.145 66.0336)
+		(width 0.2)
+		(layer "B.Cu")
+		(net "led2")
+	)
+	(segment
 		(start 97.4832 66.0654)
 		(end 97.2854 66.2632)
@@
 		(net "Net-(J1-CC2)")
 	)
-	(segment
-		(start 118.0556 64.9442)
-		(end 118.0592 64.9478)
-		(width 0.2)
-		(layer "F.Cu")
-		(net "led2")
-	)
-	(segment
-		(start 128.0414 65.405)
-		(end 127 65.405)
-		(width 0.2)
-		(layer "F.Cu")
-		(net "led2")
-	)
-	(segment
-		(start 118.0556 64.0757)
-		(end 118.0556 64.9442)
-		(width 0.2)
-		(layer "F.Cu")
-		(net "led2")
-	)
-	(segment
-		(start 127 65.405)
-		(end 126.7206 65.6844)
-		(width 0.2)
-		(layer "F.Cu")
-		(net "led2")
-	)
-	(via
-		(at 126.7206 65.6844)
-		(size 0.6)
-		(drill 0.3)
-		(layers "F.Cu" "B.Cu")
-		(net "led2")
-	)
-	(via
-		(at 118.0592 64.9478)
-		(size 0.6)
-		(drill 0.3)
-		(layers "F.Cu" "B.Cu")
-		(net "led2")
-	)
-	(segment
-		(start 126.3714 66.0336)
-		(end 126.7206 65.6844)
-		(width 0.2)
-		(layer "B.Cu")
-		(net "led2")
-	)
-	(segment
-		(start 119.145 66.0336)
-		(end 126.3714 66.0336)
-		(width 0.2)
-		(layer "B.Cu")
-		(net "led2")
-	)
-	(segment
-		(start 118.0592 64.9478)
-		(end 119.145 66.0336)
-		(width 0.2)
-		(layer "B.Cu")
-		(net "led2")
-	)
-	(segment
-		(start 105.3338 63.2992)
-		(end 105.3314 63.2968)
-		(width 0.2)
-		(layer "F.Cu")
-		(net "Net-(D1-A)")
-	)
-	(segment
-		(start 105.3338 64.3342)
-		(end 105.3338 63.2992)
-		(width 0.2)
-		(layer "F.Cu")
-		(net "Net-(D1-A)")
-	)
-	(segment
-		(start 129.0614 65.405)
-		(end 130.2028 65.405)
-		(width 0.2)
-		(layer "F.Cu")
-		(net "Net-(D2-A)")
-	)
-	(segment
-		(start 130.2028 65.405)
-		(end 130.3274 65.5296)
-		(width 0.2)
-		(layer "F.Cu")
-		(net "Net-(D2-A)")
-	)
 	(zone
